Commit message: Updating to ros kinetic

File: reactive_grasping_description/robot/vito.urdf (robot description, URDF)
Before this commit: robot vito, 61 links, 60 joints
Joints:
- removed joint right_arm_0_joint
- removed joint right_arm_0_joint_stiffness
- removed joint right_arm_1_joint
- removed joint right_arm_1_joint_stiffness
- removed joint right_arm_2_joint
- removed joint right_arm_2_joint_stiffness
- removed joint right_arm_3_joint
- removed joint right_arm_3_joint_stiffness
- removed joint right_arm_4_joint
- removed joint right_arm_4_joint_stiffness
- removed joint right_arm_5_joint
- removed joint right_arm_5_joint_stiffness
- removed joint right_arm_6_joint
- removed joint right_arm_6_joint_stiffness
- added joint right_arm_a1_joint: type revolute, parent right_arm_base_link, child right_arm_1_link, origin xyz=0 0 0.11 rpy=0 0 0, axis 0 0 1, limit lower=-2.96705972839 upper=2.96705972839 effort=176 velocity=1.91986217719
- added joint right_arm_a1_joint_stiffness: type revolute, parent right_arm_base_link, child right_arm_1_link_dummy, axis 0 0 1, limit lower=0 upper=5000 effort=0 velocity=20000
- added joint right_arm_a2_joint: type revolute, parent right_arm_1_link, child right_arm_2_link, origin xyz=0 0 0.2005 rpy=0 0 0, axis 0 -1 0, limit lower=-2.09439510239 upper=2.09439510239 effort=176 velocity=1.91986217719
- added joint right_arm_a2_joint_stiffness: type revolute, parent right_arm_1_link, child right_arm_2_link_dummy, axis 0 0 1, limit lower=0 upper=5000 effort=0 velocity=20000
- added joint right_arm_a3_joint: type revolute, parent right_arm_3_link, child right_arm_4_link, origin xyz=0 0 0.20 rpy=0 0 0, axis 0 1 0, limit lower=-2.09439510239 upper=2.09439510239 effort=100 velocity=2.23402144255
- added joint right_arm_a3_joint_stiffness: type revolute, parent right_arm_3_link, child right_arm_4_link_dummy, axis 0 0 1, limit lower=0 upper=5000 effort=0 velocity=20000
- added joint right_arm_a4_joint: type revolute, parent right_arm_4_link, child right_arm_5_link, origin xyz=0 0 0.20 rpy=0 0 0, axis 0 0 1, limit lower=-2.96705972839 upper=2.96705972839 effort=100 velocity=3.56047167407
- added joint right_arm_a4_joint_stiffness: type revolute, parent right_arm_4_link, child right_arm_5_link_dummy, axis 0 0 1, limit lower=0 upper=5000 effort=0 velocity=20000
- added joint right_arm_a5_joint: type revolute, parent right_arm_5_link, child right_arm_6_link, origin xyz=0 0 0.19 rpy=0 0 0, axis 0 -1 0, limit lower=-2.09439510239 upper=2.09439510239 effort=38 velocity=3.21140582367
- added joint right_arm_a5_joint_stiffness: type revolute, parent right_arm_5_link, child right_arm_6_link_dummy, axis 0 0 1, limit lower=0 upper=5000 effort=0 velocity=20000
- added joint right_arm_a6_joint: type revolute, parent right_arm_6_link, child right_arm_7_link, origin xyz=0 0 0.078 rpy=0 0 0, axis 0 0 1, limit lower=-2.96705972839 upper=2.96705972839 effort=38 velocity=3.21140582367
- added joint right_arm_a6_joint_stiffness: type revolute, parent right_arm_6_link, child right_arm_7_link_dummy, axis 0 0 1, limit lower=0 upper=5000 effort=0 velocity=20000
- added joint right_arm_e1_joint: type revolute, parent right_arm_2_link, child right_arm_3_link, origin xyz=0 0 0.20 rpy=0 0 0, axis 0 0 1, limit lower=-2.96705972839 upper=2.96705972839 effort=100 velocity=2.23402144255
- added joint right_arm_e1_joint_stiffness: type revolute, parent right_arm_2_link, child right_arm_3_link_dummy, axis 0 0 1, limit lower=0 upper=5000 effort=0 velocity=20000
